File: pcb/nixie.brd (EAGLE design)
At the start: 183.1 x 100 mm, 253 parts, among them IC1 STM32F100CXC, IC12 MAX603, IC2 74141N, IC3 DS3234, IC4 MAX1771, IC6 74HCT164D, IC7 DS18B20, IC8 MAX603, Q1 BUZ11BH, Q9 BSS123, U1 CC1101RTK, U2 CC1101RTK, U3 CC1101RTK, X1 BN35N61, X2 MINI-USB_4P-85-32004-10X, X3 BU-SMA-G, X4 BU-SMA-G, X5 BN35N61, X6 LFL21902MTC1A018, X7 0896BM15A0001

Commit message: some routing improvements. about to mess about with the inductor area a little
Parts:
- removed C30, C31, C32, C33, C37, C38, C39, C40, C41, C42, C43, C44, C45, C46, C47, C48, C49, C55, C56, C57, C58, C59, C60, C61, C62, C63, C64, C65, C66, C67, C68, C69, C70, C71, C72, C73, C74, C75, C76, C77, C78, C79, C80, C81, C82, C83, C84, C85, C86, C87, C88, C89, C90, C91: (no value), rcl:C0603
- removed D12, D13: BB141, diode:SOD523
- removed Q10, Q2, Q4: (no value), SparkFun:CRYSTAL-SMD-5X3
- removed R32, R33, R34, R35, R42, R43, R44, R45, R46, R47, R48, R49: (no value), rcl:R0603
- removed SV11, SV8, SV9: (no value), con-lsta:FE05-2
- removed U$18, U$19, U$20, U$22, U$23, U$24, U$4, U$5, U$6, U$7, U$9: (no value), SparkFun:C0402
- removed U$21: ADL5605, ad8345:LFCSP_VQ_16
- removed U$8: AD8345, ad8345 - Copy:TSSOP16EXP
- removed U1, U2, U3: CC1101RTK, cc1101:QFN50P400X400X90-21N
- removed X1, X5: BN35N61, con-coax:B35N61
- removed X3, X4: BU-SMA-G, con-coax:BU-SMA-G
- removed X6: LFL21902MTC1A018, ad8345:LFL21_TC
- removed X7: 0896BM15A0001, ad8345:0896BM15A0001
- added F1: PTCPTH, SparkFun:PTC
- N10, N11, N2, N3: device russian-nixies:IN-3 -> russian-nixies-mod:IN-3
- moved R12 97.0 mm to (75.1, 42.7), flipped to the bottom, turned to 180 degrees
- moved C22 18.6 mm to (18.7, 37.0)
- moved L2 10.7 mm to (49.9, 52.3), turned to 180 degrees
- moved C1 3.81 mm to (27.5, 39.1), turned to 180 degrees
- moved C16 2.77 mm to (27.9, 42.3)
- moved R13 1.40 mm to (12.7, 30.9)
- moved R8 1.14 mm to (12.7, 33.0)
- moved C19 0.99 mm to (21.0, 35.7)
- moved R5 0.76 mm to (22.4, 35.7)
- moved D10 0.25 mm to (74.3, 41.0)
- moved R7 0.16 mm to (22.2, 31.4), turned to 270 degrees
- moved C25 0.13 mm to (96.0, 32.8)
- turned D9 to 180 degrees
Connections:
- removed net +24V: C45.2, C46.2, C47.2, C48.2, C49.2, C65.2, C66.2, C67.2, C68.2, C69.2, C77.2, C78.2, C79.2, C80.2, C81.2, SV11.1, SV8.1, SV9.1, U$8.12, U$8.7, U$8.8, U1.11, U1.14, U1.15, U1.18, U1.4, U1.9, U2.11, U2.14, U2.15, U2.18, U2.4, U2.9, U3.11, U3.14, U3.15, U3.18, U3.4, U3.9
- removed net GNDA: C30.1, C31.2, C32.2, C33.1, C37.2, C39.2, C40.2, C41.1, C43.1, C45.1, C46.1, C47.1, C48.1, C49.1, C55.2, C56.2, C57.1, C58.2, C60.2, C61.2, C62.1, C63.2, C65.1, C66.1, C67.1, C68.1, C69.1, C70.2, C72.1, C73.2, C74.2, C75.2, C76.2, C77.1, C78.1, C79.1, C80.1, C81.1, C82.2, C83.2, C84.2, C85.2, C86.2, C89.1, C91.2, D12.A, D13.A, R33.2, R35.2, R42.2, R44.1, R45.1, SV11.2, SV8.2, SV9.2, U$21.P$1, U$8.10, U$8.13, U$8.14, U$8.3, U$8.4, U$8.9, U$8.EXP, U1.16, U1.19, U1.21, U2.16, U2.19, U2.21, U3.16, U3.19, U3.21, X3.2, X5.2, X6.1, X6.3, X6.5, X6.7, X7.2, X7.5, X7.6
- removed net LED_B0: IC1.41
- removed net LED_B1: IC1.40
- removed net N$103: R12.1, U1.2
- removed net N$106: R12.2, SV8.7
- removed net N$107: C40.1, C44.1, U$7.2
- removed net N$108: C38.1, U$5.2, U$6.1
- removed net N$109: C37.1, U$5.1, U1.13
- removed net N$110: C38.2, U$4.1, U1.12
- removed net N$111: C42.2, U$8.6
- removed net N$115: R42.1, U1.17
- removed net N$116: C42.1, R43.2, R44.2
- removed net N$117: C44.2, R43.1, R45.2
- removed net N$118: C43.2, U$8.5
- removed net N$119: C60.1, U$19.2, U$20.1
- removed net N$120: C61.1, C64.1, U$20.2
- removed net N$121: C59.1, U$18.2, U$19.1
- removed net N$122: C58.1, U$18.1, U2.13
- removed net N$124: D8.C, D9.C, L2.1
- removed net N$150: C59.2, U$9.1, U2.12
- removed net N$151: R33.1, U2.17
- removed net N$152: C64.2, X3.1
- removed net N$153: SV9.9
- removed net N$154: SV9.10, U2.6
- removed net N$155: C62.2, U3.5
- removed net N$156: SV11.5, U3.1
- removed net N$157: SV11.8, U3.7
- removed net N$158: SV11.6, U3.20
- removed net N$159: C70.1, C90.1, Q4.1, U3.10
- removed net N$160: C63.1, Q4.3, U3.8
- removed net N$161: R34.1, U3.2
- removed net N$162: R34.2, SV11.7
- removed net N$163: U3.12, X7.4
- removed net N$164: C74.1, C87.1, U$23.2
- removed net N$165: U3.13, X7.3
- removed net N$166: U$23.1, X7.1
- removed net N$167: C87.2, U$21.1
- removed net N$168: C71.2, X6.8
- removed net N$169: R35.1, U3.17
- removed net N$170: U$21.10, U$21.11, U$21.12, U$21.9, U$22.1, U$24.1
- removed net N$171: SV11.9, U3.3
- removed net N$172: SV11.10, U3.6
- removed net N$173: X5.1, X6.4
- removed net N$174: C71.1, C72.2, U$24.2
- removed net N$175: C73.1, C75.1, C76.1, C82.1, C83.1, C84.1, C85.1, U$21.3, U$21.4, U$22.2
- removed net N$176: C88.2, D12.C, R47.2
- removed net N$177: C86.1, U$21.2
- removed net N$178: C89.2, R46.2, R47.1
- removed net N$179: R46.1
- removed net N$180: C91.1, R48.2, R49.1
- removed net N$181: C90.2, D13.C, R48.1
- removed net N$58: C30.2, U1.5
- removed net N$59: SV9.6, U2.20
- removed net N$60: C56.1, C88.1, Q2.1, U2.10
- removed net N$61: C55.1, Q2.3, U2.8
- removed net N$62: R32.1, U2.2
- removed net N$63: R32.2, SV9.7
- removed net N$65: SV8.5, U1.1
- removed net N$70: IC1.14, Q9.1
- removed net N$72: SV8.8, U1.7
- removed net N$75: SV8.6, U1.20
- removed net N$79: C32.1, Q10.1, U1.10
- removed net N$87: C57.2, U$9.2
- removed net N$89: C31.1, Q10.3, U1.8
- removed net N$90: C33.2, U$4.2
- removed net N$93: C39.1, U$6.2, U$7.1
- net +12V: now also D8.C, D9.C; no longer D10.C, L2.2, SG2.+
- net +5V: now also D10.C, R12.2, SG2.+
- net GND: no longer X1.2, X1.3, X1.4, X1.5, X3.3, X3.4, X3.5, X4.2, X4.3, X4.4, X4.5, X5.3, X5.4, X5.5
- net N$1: now also F1.P$1, J2.3, J2.3_1; no longer C41.2, U2.5
- net N$129: now also IC1.41; no longer IC1.39
- net N$49: now also D9.A, F1.P$2; no longer SV9.5, U2.1
- net N$50: now also IC1.11; no longer SV9.8, U2.7
- net N$52: now also IC1.40, Q9.1; no longer D9.A, J2.3, J2.3_1
- net N$55: now also R12.1
Routing:
- net +24V: track 181.2 -> 0.00 mm, vias 12 -> 0
- net GNDA: track 64.5 -> 0.00 mm, vias 20 -> 0
- net N$70: track 36.7 -> 0.00 mm, vias 4 -> 0
- net +12V: track 254.3 -> 230.9 mm
- net +5V: track 67.4 -> 88.8 mm
- net N$124: track 19.9 -> 0.00 mm, vias 4 -> 0
- net N$65: track 16.6 -> 0.00 mm
- net N$157: track 14.1 -> 0.00 mm, vias 1 -> 0
- net N$75: track 12.9 -> 0.00 mm, vias 1 -> 0
- net N$72: track 10.2 -> 0.00 mm
- net N$171: track 9.93 -> 0.00 mm
- net N$175: track 9.37 -> 0.00 mm
- net N$89: track 8.84 -> 0.00 mm
- net N$79: track 8.29 -> 0.00 mm
- net N$156: track 7.57 -> 0.00 mm
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- removed copper zone on layer 16, net GNDA

Commit message: finished moving inductor
Parts:
- moved C6 9.83 mm to (36.8, 39.9)
- moved C54 7.90 mm to (38.6, 27.8)
- moved L1 6.75 mm to (44.9, 32.7)
- moved D1 6.29 mm to (35.7, 32.9)
- moved R7 1.18 mm to (21.7, 30.4), turned to 0 degrees
- moved J2 0.89 mm to (45.3, 48.8)
- moved IC2 0.76 mm to (11.9, 39.1)
- moved C5 0.65 mm to (42.5, 28.8)
- moved Q1 0.52 mm to (28.5, 35.6)
- moved R13 0.51 mm to (12.2, 30.9)
- moved R8 0.51 mm to (12.2, 33.0)
- moved C7 0.38 mm to (13.5, 40.4)
- moved R5 0.38 mm to (22.0, 35.7)
- moved C19 0.38 mm to (20.6, 35.7)
- moved R31 0.18 mm to (38.8, 8.12)
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Routing:
- net GND: track 358.3 -> 346.2 mm
- net N$26: track 49.2 -> 39.1 mm
- net N$15: track 17.1 -> 24.4 mm
- net N$20: track 3.48 -> 8.12 mm
- net +12V: track 230.9 -> 234.3 mm
- net GND1: track 218.0 -> 214.9 mm
- net N$129: track 73.2 -> 75.6 mm
- net N$14: track 10.3 -> 12.1 mm
- net N$21: track 16.2 -> 17.5 mm
- net N$11: track 78.1 -> 79.3 mm
- net +5V: track 88.8 -> 89.8 mm
- net N$6: track 96.5 -> 97.3 mm
- net N$100: track 12.6 -> 11.8 mm
- net N$105: track 7.50 -> 6.74 mm
- net N$102: track 26.0 -> 25.2 mm
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
Commit message: mostly silk screen stuff
Parts:
- moved D1 1.09 mm to (36.6, 33.5), turned to 240 degrees
- moved C6 0.89 mm to (36.8, 40.8)
- moved C54 0.76 mm to (37.8, 27.8)
- moved R4 0.13 mm to (31.8, 34.7)
Routing:
- net +12V: track 234.3 -> 240.1 mm
- net GND: track 346.2 -> 341.3 mm, vias 81 -> 91
- net N$26: track 39.1 -> 41.2 mm
- net DIGITS7: track 166.7 -> 165.8 mm
Other:
- board text added: "M. BREJZA"
- board text added: "MAY 13"
- board text added: "PROG"
- board text added: "RUN"
- board text added: "SWD"
- board text added: "label positions"
- board text added: "make sure diodes correct package"

Commit message: almost done
Parts:
- removed S6: (no value), SparkFun:TACTILE-PTH
- added S1, S3: (no value), Mine:TACTSIDE
- C1, C10, C11, C12, C13, C14, C15, C18, C20, C21, C22, C25, C26, C27, C35, C36, C4, C52, C53, C7, C8, C9, C93: value (none) -> 100n
- C16, C17, C28, C29, C92: value (none) -> 10u
- C2, C23, C3, C34, C5, Q3, R12, R51, R9: value (none) -> nc
- C24: value (none) -> 100n; device rcl:C1206 -> rcl:C0603
- C50, C51: value (none) -> 1u
- C54, L1: value (none) -> 100u
- C6: value (none) -> 2.2u 250V
- D10, D11, D8, D9: value CGRM4001-G -> (none); device diode:SOD-123_MINI-SMA -> diode:SOD123
- D2, D3, D4, D5, D6, D7: value CGRM4001-G -> 1n4148
- R1, R36, R37, R50, R6: value (none) -> 10k
- R13, R8: value (none) -> 22k
- R14, R16, R18, R20, R22, R24: value (none) -> 1M
- R15, R17, R19, R21, R23, R25: value (none) -> 47k
- R2: value (none) -> 100
- R3: value (none) -> 1k
- R30, R31: value (none) -> tbc
- R38: value (none) -> 220k
- R39, R40, R41: value (none) -> 200k
- R4: value (none) -> 0.05
- R5: value (none) -> 1M5
- R7: value (none) -> 4k7 trim
- S2, S4, S5: device SparkFun:TACTILE-PTH -> Mine:TACTSIDE
- T1, T11, T13, T14, T3, T5, T7, T9: value (none) -> pnphv
- T10, T12, T2, T4, T6, T8: value (none) -> npnhvsmd
- T21, T22: value (none) -> npnhvth
- moved S2 25.3 mm to (54.7, 30.0)
- moved C24 3.05 mm to (58.8, 34.4), flipped to the bottom, turned to 270 degrees
- moved S4 1.91 mm to (72.8, 30.0)
- moved S5 1.71 mm to (63.8, 30.0)
- moved U$1 0.89 mm to (89.7, 27.4)
- moved C20 0.38 mm to (86.1, 32.5)
- moved C92 0.38 mm to (84.8, 32.5)
Connections:
- net +3V3: now also S3.1; no longer S2.2, S4.2, S5.2, S6.1, S6.2
- net BUT0: now also S5.2; no longer S5.3, S5.4
- net BUT1: now also S2.2; no longer S6.3, S6.4
- net BUT2: now also S4.2; no longer S4.3, S4.4
- net BUT3: now also S3.2; no longer S2.3, S2.4
Routing:
- net +3V3: track 203.0 -> 235.8 mm
- net GND: track 341.3 -> 333.1 mm, vias 91 -> 92
- net BUT2: track 32.0 -> 24.3 mm
- net BUT0: track 34.0 -> 26.8 mm
- net BUT1: track 42.0 -> 35.3 mm
- net BUT3: track 22.6 -> 16.9 mm
- net SWD_DIO: track 30.5 -> 33.0 mm, vias 1 -> 3
- net N$21: track 17.5 -> 15.8 mm
- net N$64: track 9.76 -> 8.36 mm, vias 1 -> 0
- net +12V: track 240.1 -> 241.3 mm, vias 12 -> 10
- net N$7: track 28.9 -> 28.0 mm
- net N$131: track 5.09 -> 4.20 mm
- net IR: track 30.8 -> 30.1 mm
- net N$94: track 16.6 -> 16.0 mm
- net N$12: track 82.5 -> 81.9 mm
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
Commit message: just before merge
Parts:
- moved SJ2 6.66 mm to (80.5, 43.1), flipped to the bottom, turned to 90 degrees
- moved C50 0.51 mm to (112.8, 6.10)
- moved R12 0.28 mm to (74.8, 42.8)
- moved D9 0.25 mm to (50.4, 43.2)
- moved R13 0.13 mm to (12.1, 30.9)
- moved R8 0.13 mm to (12.1, 33.0)
- moved U$1 0.13 mm to (89.8, 27.4)
Routing:
- net +3V3: track 235.8 -> 226.5 mm
- net N$51: track 2.78 -> 5.23 mm, vias 0 -> 1
- net HV2_B: track 12.5 -> 11.2 mm
- net +5V: track 89.8 -> 90.4 mm
- net BUT3: track 16.9 -> 16.3 mm
- net IR: track 30.1 -> 29.6 mm
- net N$144: track 1.52 -> 2.03 mm
- net GND: track 333.1 -> 332.8 mm, vias 92 -> 98
Other:
- board text added: "+"
- board text added: "-"
- board text added: "0V"
- board text added: "5-12V"
- board text added: "C"
- board text added: "D"
- board text added: "RX"
- board text added: "TX"

Commit message: deleted stuff for merging
Parts:
- removed C23: nc, rcl:C0603
- removed C93: 100n, rcl:C0603
- removed L2: (no value), wuerth-elektronik:0805
- removed R9: nc, rcl:R0805
- removed S1: (no value), Mine:TACTSIDE
- removed SV6: (no value), Mine:EDGE_6
Connections:
- removed net RXD: SV6.2
- removed net TXD: SV6.3
- net GND: no longer C93.1
- net VBAT: no longer C93.2
Other:
- board text removed: "label positions"
- board text removed: "make sure diodes correct package"
- board text removed: "move header down a bit ->"
Changed lines of the file:
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@@
 <wire x1="118.872" y1="-36.576" x2="105.41" y2="-36.576" width="0.254" layer="51"/>
 <wire x1="133.858" y1="-36.83" x2="119.634" y2="-36.83" width="0.254" layer="51"/>
-<wire x1="47.752" y1="-36.322" x2="34.798" y2="-36.322" width="0" layer="19"/>
-<wire x1="65.532" y1="-33.528" x2="58.42" y2="-33.528" width="0" layer="19"/>
-<wire x1="89.408" y1="-32.512" x2="79.502" y2="-32.512" width="0" layer="19"/>
-<wire x1="109.22" y1="-30.48" x2="100.33" y2="-30.48" width="0" layer="19"/>
-<wire x1="100.33" y1="-30.48" x2="100.33" y2="-27.178" width="0" layer="19"/>
-<wire x1="116.84" y1="-25.654" x2="113.792" y2="-25.654" width="0" layer="19"/>
-<wire x1="52.578" y1="-27.178" x2="46.482" y2="-27.178" width="0" layer="19"/>
-<wire x1="100.33" y1="-27.178" x2="91.186" y2="-27.178" width="0" layer="19"/>
-<wire x1="138.176" y1="-26.924" x2="120.142" y2="-26.924" width="0" layer="19"/>
 <wire x1="0" y1="24.892" x2="128.016" y2="24.892" width="0" layer="20"/>
 <wire x1="128.016" y1="24.892" x2="128.016" y2="0" width="0" layer="20"/>
@@
 <circle x="13.462" y="-16.764" radius="8.636" width="0" layer="16"/>
 <circle x="34.798" y="-17.018" radius="8.636" width="0" layer="16"/>
-<circle x="25.4" y="-10.668" radius="3.048" width="0" layer="16"/>
 <circle x="58.166" y="-17.526" radius="8.636" width="0" layer="16"/>
 <circle x="79.502" y="-17.78" radius="8.636" width="0" layer="16"/>
-<circle x="70.612" y="-12.954" radius="3.048" width="0" layer="16"/>
 <circle x="91.186" y="-17.78" radius="3.048" width="0" layer="16"/>
 <circle x="100.33" y="-18.288" radius="6.1012" width="0" layer="16"/>
@@
 <circle x="124.714" y="28.702" radius="2.54" width="0.254" layer="51"/>
 <circle x="118.872" y="46.863" radius="2.54" width="0.254" layer="51"/>
-<text x="-45.085" y="18.669" size="1.778" layer="21">move header down a bit -&gt;</text>
-<rectangle x1="119.253" y1="61.341" x2="159.258" y2="81.407" layer="16"/>
-<rectangle x1="129.286" y1="71.628" x2="149.352" y2="111.76" layer="16" rot="R90"/>
-<rectangle x1="96.5835" y1="58.8645" x2="116.6495" y2="83.8835" layer="16" rot="R90"/>
-<rectangle x1="-7.757" y1="5.054" x2="1.583" y2="5.344" layer="1" rot="R180"/>
-<rectangle x1="-9.345" y1="13.335" x2="-4.445" y2="13.845" layer="1"/>
-<rectangle x1="0.503" y1="-19.309" x2="13.483" y2="-6.269" layer="16"/>
-<rectangle x1="130.586" y1="-4.983" x2="135.566" y2="0.057" layer="1"/>
-<rectangle x1="151.5809" y1="10.5981" x2="153.9811" y2="11.8681" layer="1" rot="R90"/>
-<rectangle x1="151.892" y1="8.89" x2="157.988" y2="10.922" layer="1" rot="R270"/>
 <hole x="19.812" y="46.482" drill="3.2"/>
 <hole x="3.81" y="29.21" drill="3.2"/>
@@
 <text x="13.716" y="3.429" size="1.4224" layer="122" ratio="15" rot="MR0">M. BREJZA</text>
 <text x="13.716" y="1.524" size="1.4224" layer="122" ratio="15" rot="MR0">MAY 13</text>
-<text x="66.294" y="50.927" size="1.4224" layer="122" ratio="15" rot="R90">make sure diodes correct package</text>
 <text x="76.962" y="46.101" size="1.4224" layer="121" ratio="15" rot="R90">SWD</text>
-<text x="89.154" y="51.308" size="1.4224" layer="121" ratio="15">label positions</text>
 <text x="102.743" y="44.958" size="1.016" layer="121" ratio="15" rot="R90">RUN</text>
 <text x="91.313" y="44.577" size="1.016" layer="121" ratio="15" rot="R90">PROG</text>
@@
 <rectangle x1="4.835" y1="8.055" x2="5.015" y2="8.065" layer="201"/>
 <rectangle x1="4.865" y1="8.065" x2="4.965" y2="8.075" layer="201"/>
-<rectangle x1="-3.048" y1="-3.048" x2="0" y2="0" layer="1"/>
 <text x="86.233" y="46.355" size="1.27" layer="121" ratio="15" rot="R270">D</text>
 <text x="82.423" y="45.339" size="1.27" layer="121" ratio="15" rot="R90">C</text>
-<text x="85.09" y="52.07" size="1.4224" layer="121" ratio="15">-</text>
 <text x="77.216" y="46.228" size="1.4224" layer="121" ratio="15">+</text>
 <text x="85.09" y="44.069" size="1.27" layer="121" ratio="15" rot="R90">0V</text>
 <text x="108.331" y="44.069" size="1.27" layer="121" ratio="15" rot="R90">TX</text>
 <text x="104.394" y="44.069" size="1.27" layer="122" ratio="15" rot="MR90">RX</text>
-<text x="111.633" y="53.086" size="1.27" layer="121" ratio="15" rot="R180">0V</text>
 <text x="114.681" y="45.085" size="1.4224" layer="122" ratio="15">-</text>
 <wire x1="89.789" y1="50.038" x2="89.789" y2="42.926" width="0.4064" layer="121"/>
@@
 </element>
 <element name="SV4" library="Mine" package="EDGE_10" value="" x="112.649" y="49.911"/>
-<element name="SV6" library="Mine" package="EDGE_6" value="" x="96.012" y="61.087"/>
 <element name="IC12" library="Mine" package="SO08" value="MAX603" x="53.848" y="36.195" rot="MR180"/>
 <element name="C28" library="rcl" package="C0603" value="10u" x="57.15" y="37.973" rot="MR270"/>
@@
 <element name="D8" library="diode" package="SOD123" value="" x="65.405" y="47.879" rot="MR180"/>
 <element name="D9" library="diode" package="SOD123" value="" x="50.419" y="43.18" rot="MR180"/>
-<element name="L2" library="wuerth-elektronik" package="0805" value="" x="49.911" y="52.324" rot="MR180"/>
 <element name="C34" library="rcl" package="SMC_C" value="nc" x="48.133" y="34.798" rot="MR90"/>
 <element name="C35" library="rcl" package="C0603" value="100n" x="68.453" y="34.544" rot="MR270"/>
@@
 <element name="R1" library="rcl" package="R0603" value="10k" x="96.266" y="43.053" rot="MR180"/>
 <element name="SJ2" library="SparkFun" package="SJ_2S-NO" value="SOLDERJUMPERNO" x="80.518" y="43.053" rot="MR90"/>
-<element name="C23" library="rcl" package="C0603" value="nc" x="91.313" y="63.5" rot="MR90"/>
-<element name="R9" library="rcl" package="R0805" value="nc" x="89.027" y="63.246" rot="MR270"/>
 <element name="U$1" library="Mine" package="IRREC" value="IRREC" x="89.789" y="27.432"/>
 <element name="SV7" library="Mine" package="EDGE_4" value="" x="83.058" y="48.133"/>
@@
 <element name="R51" library="rcl" package="R0603" value="nc" x="87.63" y="45.466" rot="MR90"/>
 <element name="C92" library="rcl" package="C0603" value="10u" x="84.836" y="32.512" rot="MR270"/>
-<element name="C93" library="rcl" package="C0603" value="100n" x="82.296" y="53.594" rot="MR180"/>
 <element name="SJ3" library="SparkFun" package="SJ_2S-NO" value="SOLDERJUMPERNO" x="83.82" y="40.767" rot="MR90"/>
 <element name="F1" library="SparkFun" package="PTC" value="PTCPTH" x="53.848" y="46.101" rot="R270"/>
 <element name="R12" library="rcl" package="R0603" value="nc" x="74.803" y="42.799" rot="MR180"/>
-<element name="S1" library="Mine" package="TACTSIDE" value="" x="-50.292" y="-44.45"/>
 <element name="S2" library="Mine" package="TACTSIDE" value="" x="54.737" y="29.972"/>
 <element name="S3" library="Mine" package="TACTSIDE" value="" x="81.788" y="29.972"/>
@@
 <contactref element="U$3" pad="2A"/>
 <contactref element="R50" pad="2"/>
-<contactref element="C93" pad="1"/>
 <contactref element="C92" pad="2"/>
 <via x="98.171" y="40.513" extent="1-16" drill="0.381" shape="octagon"/>
@@
 <via x="57.15" y="40.132" extent="1-16" drill="0.381" shape="octagon"/>
 <via x="53.848" y="38.989" extent="1-16" drill="0.381" shape="octagon"/>
-<wire x1="84.201" y1="49.022" x2="81.446" y2="53.594" width="0" layer="19" extent="16-16"/>
 </signal>
 <signal name="+5V">
@@
 <wire x1="94.107" y1="42.672" x2="92.837" y2="43.942" width="0.254" layer="1"/>
 </signal>
-<signal name="RXD">
-<contactref element="SV6" pad="2"/>
-</signal>
-<signal name="TXD">
-<contactref element="SV6" pad="3"/>
-</signal>
 <signal name="N$66">
 <contactref element="T22" pad="B"/>
@@
 <wire x1="85.217" y1="40.767" x2="85.598" y2="40.4622" width="0.254" layer="16"/>
 <via x="85.217" y="40.767" extent="1-16" drill="0.381" diameter="0.8128" shape="octagon"/>
-<contactref element="C93" pad="2"/>
 <contactref element="SJ3" pad="2"/>
 <wire x1="83.82" y1="41.217" x2="84.767" y2="41.217" width="0.4064" layer="16"/>
 <wire x1="84.767" y1="41.217" x2="85.217" y2="40.767" width="0.4064" layer="16"/>
-<wire x1="83.82" y1="41.217" x2="83.146" y2="53.594" width="0" layer="19" extent="16-16"/>
 </signal>
 <signal name="N$3">

Commit message: off for fab
Routing:
- net N$58: track 0.00 -> 23.0 mm
- net N$60: track 0.00 -> 9.80 mm
- net N$59: track 0.00 -> 3.50 mm
- net VPP: track 150.9 -> 148.9 mm
- net N$2: track 82.8 -> 80.8 mm
- net N$19: track 10.3 -> 9.18 mm
- net LED5: track 13.5 -> 12.7 mm
- net DIGITS0: track 187.4 -> 186.8 mm
Other:
- board size 183.1 x 100 mm -> 128 x 50 mm
- board text added: "Rev. 1"
