File: pcb/nixie.sch (EAGLE design)
At the start: 253 parts, among them IC1 STM32F100CXC, IC12 MAX603, IC2 74141N, IC3 DS3234, IC4 MAX1771, IC6 74HCT164D, IC7 DS18B20, IC8 MAX603, Q1 BUZ11BH, Q9 BSS123, U1 CC1101RTK, U2 CC1101RTK, U3 CC1101RTK, X1 BN35N61, X2 MINI-USB_4P-85-32004-10X, X3 BU-SMA-G, X4 BU-SMA-G, X5 BN35N61, X6 LFL21902MTC1A018, X7 0896BM15A0001

Commit message: some routing improvements. about to mess about with the inductor area a little
Parts:
- removed C30, C31, C32, C33, C37, C38, C39, C40, C41, C42, C43, C44, C45, C46, C47, C48, C49, C55, C56, C57, C58, C59, C60, C61, C62, C63, C64, C65, C66, C67, C68, C69, C70, C71, C72, C73, C74, C75, C76, C77, C78, C79, C80, C81, C82, C83, C84, C85, C86, C87, C88, C89, C90, C91: (no value), rcl:C-EUC0603
- removed D12, D13: BB141, diode:BB141
- removed Q10, Q2, Q4: (no value), SparkFun:CRYSTAL5X3
- removed R32, R33, R34, R35, R42, R43, R44, R45, R46, R47, R48, R49: (no value), rcl:R-EU_R0603
- removed SV11, SV8, SV9: (no value), con-lsta:FE05-2
- removed U$18, U$19, U$20, U$22, U$23, U$24, U$4, U$5, U$6, U$7, U$9: (no value), SparkFun:INDUCTOR0402
- removed U$21: ADL5605, ad8345:ADL5605
- removed U$8: AD8345, ad8345 - Copy:AD8345
- removed U1, U2, U3: CC1101RTK, cc1101:CC1101RTK
- removed X1, X5: BN35N61, con-coax:BN35N61
- removed X3, X4: BU-SMA-G, con-coax:BU-SMA-G
- removed X6: LFL21902MTC1A018, ad8345:LFL21902MTC1A018
- removed X7: 0896BM15A0001, ad8345:0896BM15A0001
- added F1: PTCPTH, SparkFun:PTCPTH
- N10, N11, N2, N3: device russian-nixies:IN-3 -> russian-nixies-mod:IN-3
Connections:
- removed net +24V: C45.2, C46.2, C47.2, C48.2, C49.2, C65.2, C66.2, C67.2, C68.2, C69.2, C77.2, C78.2, C79.2, C80.2, C81.2, SV11.1, SV8.1, SV9.1, U$8.ENBL, U$8.VPS1, U$8.VPS2, U1.AVDD, U1.AVDD_2, U1.AVDD_3, U1.AVDD_4, U1.DGUARD, U1.DVDD, U2.AVDD, U2.AVDD_2, U2.AVDD_3, U2.AVDD_4, U2.DGUARD, U2.DVDD, U3.AVDD, U3.AVDD_2, U3.AVDD_3, U3.AVDD_4, U3.DGUARD, U3.DVDD
- removed net GNDA: C30.1, C31.2, C32.2, C33.1, C37.2, C39.2, C40.2, C41.1, C43.1, C45.1, C46.1, C47.1, C48.1, C49.1, C55.2, C56.2, C57.1, C58.2, C60.2, C61.2, C62.1, C63.2, C65.1, C66.1, C67.1, C68.1, C69.1, C70.2, C72.1, C73.2, C74.2, C75.2, C76.2, C77.1, C78.1, C79.1, C80.1, C81.1, C82.2, C83.2, C84.2, C85.2, C86.2, C89.1, C91.2, D12.A, D13.A, R33.2, R35.2, R42.2, R44.1, R45.1, SV11.2, SV8.2, SV9.2, U$21.GND, U$8.COM1, U$8.COM2, U$8.COM3_1, U$8.COM3_2, U$8.COM3_3, U$8.COM3_4, U$8.EP, U1.EP, U1.GND, U1.GND_2, U2.EP, U2.GND, U2.GND_2, U3.EP, U3.GND, U3.GND_2, X3G1.GND, X5G$1.GND, X6.GND, X6.GND1, X6.GND2, X6.GND3, X7.GND, X7.GND1, X7.GND2
- removed net LED_B0: IC1.PB5
- removed net LED_B1: IC1.PB4
- removed net N$103: R12.1, U1.SO(GDO1)
- removed net N$106: R12.2, SV8.7
- removed net N$107: C40.1, C44.1, U$7.2
- removed net N$108: C38.1, U$5.2, U$6.1
- removed net N$109: C37.1, U$5.1, U1.RF_N
- removed net N$110: C38.2, U$4.1, U1.RF_P
- removed net N$111: C42.2, U$8.LOIP
- removed net N$115: R42.1, U1.RBIAS
- removed net N$116: C42.1, R43.2, R44.2
- removed net N$117: C44.2, R43.1, R45.2
- removed net N$118: C43.2, U$8.LOIN
- removed net N$119: C60.1, U$19.2, U$20.1
- removed net N$120: C61.1, C64.1, U$20.2
- removed net N$121: C59.1, U$18.2, U$19.1
- removed net N$122: C58.1, U$18.1, U2.RF_N
- removed net N$124: D8.C, D9.C, L2.1
- removed net N$150: C59.2, U$9.1, U2.RF_P
- removed net N$151: R33.1, U2.RBIAS
- removed net N$152: C64.2, X3G1.1
- removed net N$153: SV9.9
- removed net N$154: SV9.10, U2.GDO0(ATEST)
- removed net N$155: C62.2, U3.DCOUPL
- removed net N$156: SV11.5, U3.SCLK
- removed net N$157: SV11.8, U3.CSN
- removed net N$158: SV11.6, U3.SI
- removed net N$159: C70.1, C90.1, Q4.1, U3.XOSC_Q2
- removed net N$160: C63.1, Q4.2, U3.XOSC_Q1
- removed net N$161: R34.1, U3.SO(GDO1)
- removed net N$162: R34.2, SV11.7
- removed net N$163: U3.RF_P, X7.BAL2
- removed net N$164: C74.1, C87.1, U$23.2
- removed net N$165: U3.RF_N, X7.BAL1
- removed net N$166: U$23.1, X7.UN
- removed net N$167: C87.2, U$21.RFIN
- removed net N$168: C71.2, X6.IN
- removed net N$169: R35.1, U3.RBIAS
- removed net N$170: U$21.RFOUT, U$21.RFOUT1, U$21.RFOUT2, U$21.RFOUT3, U$22.1, U$24.1
- removed net N$171: SV11.9, U3.GDO2
- removed net N$172: SV11.10, U3.GDO0(ATEST)
- removed net N$173: X5G$1.1, X6.OUT
- removed net N$174: C71.1, C72.2, U$24.2
- removed net N$175: C73.1, C75.1, C76.1, C82.1, C83.1, C84.1, C85.1, U$21.VBIAS, U$21.VCC, U$22.2
- removed net N$176: C88.2, D12.C, R47.2
- removed net N$177: C86.1, U$21.DISABLE
- removed net N$178: C89.2, R46.2, R47.1
- removed net N$179: R46.1
- removed net N$180: C91.1, R48.2, R49.1
- removed net N$181: C90.2, D13.C, R48.1
- removed net N$58: C30.2, U1.DCOUPL
- removed net N$59: SV9.6, U2.SI
- removed net N$60: C56.1, C88.1, Q2.1, U2.XOSC_Q2
- removed net N$61: C55.1, Q2.2, U2.XOSC_Q1
- removed net N$62: R32.1, U2.SO(GDO1)
- removed net N$63: R32.2, SV9.7
- removed net N$65: SV8.5, U1.SCLK
- removed net N$70: IC1.PA4, Q9.G
- removed net N$72: SV8.8, U1.CSN
- removed net N$75: SV8.6, U1.SI
- removed net N$79: C32.1, Q10.1, U1.XOSC_Q2
- removed net N$87: C57.2, U$9.2
- removed net N$89: C31.1, Q10.2, U1.XOSC_Q1
- removed net N$90: C33.2, U$4.2
- removed net N$93: C39.1, U$6.2, U$7.1
- net +12V: now also D8.C, D9.C; no longer D10.C, L2.2, SG2.1
- net +5V: now also D10.C, R12.2, SG2.1
- net N$1: now also F1.1, J2.3, J2.4; no longer C41.2, U2.DCOUPL
- net N$129: now also IC1.PB5; no longer IC1.PB3
- net N$49: now also D9.A, F1.2; no longer SV9.5, U2.SCLK
- net N$50: now also IC1.PA1; no longer SV9.8, U2.CSN
- net N$52: now also IC1.PB4, Q9.G; no longer D9.A, J2.3, J2.4
- net N$55: now also R12.1
Other:
- moved on the sheet: D9, J2, L2, R12

Commit message: mostly silk screen stuff
Other:
- moved on the sheet: C28, C29
Changed lines of the file:
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@@
 <instance part="SV6" gate="G$1" x="287.02" y="-27.94"/>
 <instance part="IC12" gate="G$1" x="-40.64" y="147.32"/>
-<instance part="C28" gate="G$1" x="-58.42" y="139.7"/>
-<instance part="C29" gate="G$1" x="-20.32" y="142.24"/>
+<instance part="C28" gate="G$1" x="-55.88" y="139.7"/>
+<instance part="C29" gate="G$1" x="-20.32" y="144.78"/>
 <instance part="GND20" gate="1" x="-40.64" y="132.08"/>
 <instance part="+3V6" gate="G$1" x="-17.78" y="152.4" rot="R270"/>
@@
 </segment>
 <segment>
-<wire x1="-20.32" y1="137.16" x2="-20.32" y2="134.62" width="0.1524" layer="91"/>
+<wire x1="-20.32" y1="139.7" x2="-20.32" y2="134.62" width="0.1524" layer="91"/>
 <wire x1="-20.32" y1="134.62" x2="-35.56" y2="134.62" width="0.1524" layer="91"/>
 <wire x1="-35.56" y1="134.62" x2="-38.1" y2="134.62" width="0.1524" layer="91"/>
 <wire x1="-38.1" y1="134.62" x2="-40.64" y2="134.62" width="0.1524" layer="91"/>
 <wire x1="-40.64" y1="134.62" x2="-43.18" y2="134.62" width="0.1524" layer="91"/>
-<wire x1="-43.18" y1="134.62" x2="-58.42" y2="134.62" width="0.1524" layer="91"/>
+<wire x1="-43.18" y1="134.62" x2="-55.88" y2="134.62" width="0.1524" layer="91"/>
 <junction x="-40.64" y="134.62"/>
 <junction x="-35.56" y="134.62"/>
@@
 <segment>
 <wire x1="-22.86" y1="152.4" x2="-20.32" y2="152.4" width="0.1524" layer="91"/>
-<wire x1="-20.32" y1="152.4" x2="-20.32" y2="144.78" width="0.1524" layer="91"/>
-<wire x1="-20.32" y1="144.78" x2="-22.86" y2="144.78" width="0.1524" layer="91"/>
-<wire x1="-22.86" y1="144.78" x2="-22.86" y2="147.32" width="0.1524" layer="91"/>
-<junction x="-20.32" y="144.78"/>
+<wire x1="-20.32" y1="152.4" x2="-20.32" y2="147.32" width="0.1524" layer="91"/>
+<wire x1="-20.32" y1="147.32" x2="-22.86" y2="147.32" width="0.1524" layer="91"/>
+<junction x="-20.32" y="147.32"/>
 <junction x="-20.32" y="152.4"/>
 <pinref part="IC12" gate="G$1" pin="OUT"/>
@@
 <wire x1="-43.18" y1="213.36" x2="-55.88" y2="213.36" width="0.1524" layer="91"/>
 <wire x1="-55.88" y1="190.5" x2="-60.96" y2="190.5" width="0.1524" layer="91"/>
-<wire x1="-58.42" y1="142.24" x2="-55.88" y2="142.24" width="0.1524" layer="91"/>
 <wire x1="-55.88" y1="142.24" x2="-55.88" y2="147.32" width="0.1524" layer="91"/>
 <wire x1="-55.88" y1="147.32" x2="-55.88" y2="152.4" width="0.1524" layer="91"/>
@@
 <net name="N$136" class="0">
 <segment>
-<wire x1="345.44" y1="388.62" x2="345.44" y2="391.16" width="0.1524" layer="91"/>
 <wire x1="345.44" y1="391.16" x2="345.44" y2="424.18" width="0.1524" layer="91"/>
 <wire x1="327.66" y1="391.16" x2="345.44" y2="391.16" width="0.1524" layer="91"/>
@@
 <net name="N$139" class="0">
 <segment>
-<wire x1="350.52" y1="375.92" x2="350.52" y2="378.46" width="0.1524" layer="91"/>
 <wire x1="350.52" y1="378.46" x2="350.52" y2="424.18" width="0.1524" layer="91"/>
 <wire x1="327.66" y1="378.46" x2="350.52" y2="378.46" width="0.1524" layer="91"/>
@@
 <net name="N$142" class="0">
 <segment>
-<wire x1="355.6" y1="363.22" x2="355.6" y2="365.76" width="0.1524" layer="91"/>
 <wire x1="355.6" y1="365.76" x2="355.6" y2="424.18" width="0.1524" layer="91"/>
 <wire x1="327.66" y1="365.76" x2="355.6" y2="365.76" width="0.1524" layer="91"/>
@@
 <segment>
 <wire x1="167.64" y1="375.92" x2="157.48" y2="375.92" width="0.1524" layer="91"/>
-<wire x1="157.48" y1="375.92" x2="157.48" y2="401.32" width="0.1524" layer="91"/>
-<wire x1="157.48" y1="401.32" x2="276.86" y2="401.32" width="0.1524" layer="91"/>
-<wire x1="276.86" y1="401.32" x2="276.86" y2="386.08" width="0.1524" layer="91"/>
+<wire x1="157.48" y1="375.92" x2="157.48" y2="406.4" width="0.1524" layer="91"/>
+<wire x1="157.48" y1="406.4" x2="276.86" y2="406.4" width="0.1524" layer="91"/>
+<wire x1="276.86" y1="406.4" x2="276.86" y2="386.08" width="0.1524" layer="91"/>
 <wire x1="276.86" y1="386.08" x2="284.48" y2="386.08" width="0.1524" layer="91"/>
 <pinref part="U$10" gate="G$1" pin="SDTO"/>
@@
 <segment>
 <wire x1="167.64" y1="373.38" x2="154.94" y2="373.38" width="0.1524" layer="91"/>
-<wire x1="154.94" y1="373.38" x2="154.94" y2="403.86" width="0.1524" layer="91"/>
-<wire x1="154.94" y1="403.86" x2="274.32" y2="403.86" width="0.1524" layer="91"/>
+<wire x1="154.94" y1="373.38" x2="154.94" y2="408.94" width="0.1524" layer="91"/>
+<wire x1="154.94" y1="408.94" x2="274.32" y2="408.94" width="0.1524" layer="91"/>
 <wire x1="284.48" y1="383.54" x2="274.32" y2="383.54" width="0.1524" layer="91"/>
-<wire x1="274.32" y1="403.86" x2="274.32" y2="383.54" width="0.1524" layer="91"/>
+<wire x1="274.32" y1="408.94" x2="274.32" y2="383.54" width="0.1524" layer="91"/>
 <pinref part="U$10" gate="G$1" pin="SCKO"/>
 <pinref part="U$11" gate="G$1" pin="SCKI"/>

Commit message: almost done
Parts:
- removed S6: (no value), SparkFun:TAC_SWITCHPTH
- added S1, S3: (no value), Mine:TAC_SWITCH
- C1, C10, C11, C12, C13, C14, C15, C18, C20, C21, C22, C25, C26, C27, C35, C36, C4, C52, C53, C7, C8, C9, C93: value (none) -> 100n
- C16, C17, C28, C29, C92: value (none) -> 10u
- C2, C23, C3, C34, C5, Q3, R12, R51, R9: value (none) -> nc
- C24: value (none) -> 100n; device rcl:C-EUC1206 -> rcl:C-EUC0603
- C50, C51: value (none) -> 1u
- C54, L1: value (none) -> 100u
- C6: value (none) -> 2.2u 250V
- D10, D11, D8, D9: value CGRM4001-G -> (none); device diode:CGRM4001-G -> diode:DIODE-SOD123
- D2, D3, D4, D5, D6, D7: value CGRM4001-G -> 1n4148
- R1, R36, R37, R50, R6: value (none) -> 10k
- R13, R8: value (none) -> 22k
- R14, R16, R18, R20, R22, R24: value (none) -> 1M
- R15, R17, R19, R21, R23, R25: value (none) -> 47k
- R2: value (none) -> 100
- R3: value (none) -> 1k
- R30, R31: value (none) -> tbc
- R38: value (none) -> 220k
- R39, R40, R41: value (none) -> 200k
- R4: value (none) -> 0.05
- R5: value (none) -> 1M5
- R7: value (none) -> 4k7 trim
- S2, S4, S5: device SparkFun:TAC_SWITCHPTH -> Mine:TAC_SWITCH
- T1, T11, T13, T14, T3, T5, T7, T9: value (none) -> pnphv
- T10, T12, T2, T4, T6, T8: value (none) -> npnhvsmd
- T21, T22: value (none) -> npnhvth
Connections:
- net +3V3: now also S3.1; no longer S2.2, S4.2, S5.2, S6.1, S6.2
- net BUT0: now also S5.2; no longer S5.3, S5.4
- net BUT1: now also S2.2; no longer S6.3, S6.4
- net BUT2: now also S4.2; no longer S4.3, S4.4
- net BUT3: now also S3.2; no longer S2.3, S2.4
Other:
- note added: "nc"
- note added: "tbc"

Commit message: deleted stuff for merging
Parts:
- removed C23: nc, rcl:C-EUC0603
- removed C93: 100n, rcl:C-EUC0603
- removed L2: (no value), wuerth-elektronik:WE-CBF_0805
- removed R9: nc, rcl:R-EU_R0805
- removed S1: (no value), Mine:TAC_SWITCH
- removed SV6: (no value), Mine:FE06-1ED
Connections:
- removed net RXD: SV6.2
- removed net TXD: SV6.3
- net GND: no longer C93.1
- net VBAT: no longer C93.2
Changed lines of the file:
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@@
 <part name="Q3" library="crystal" deviceset="CRYSTAL" device="CTS406" value="nc"/>
 <part name="SV4" library="Mine" deviceset="FE05-2W" device="ED"/>
-<part name="SV6" library="Mine" deviceset="FE06-1" device="ED"/>
 <part name="IC12" library="Mine" deviceset="MAX603" device=""/>
 <part name="C28" library="rcl" deviceset="C-EU" device="C0603" value="10u"/>
@@
 <part name="D8" library="diode" deviceset="DIODE-" device="SOD123"/>
 <part name="D9" library="diode" deviceset="DIODE-" device="SOD123"/>
-<part name="L2" library="wuerth-elektronik" deviceset="WE-CBF" device="_0805"/>
 <part name="C34" library="rcl" deviceset="CPOL-EU" device="SMCC" value="nc"/>
 <part name="GND9" library="supply1" deviceset="GND" device=""/>
@@
 <part name="R1" library="rcl" deviceset="R-EU_" device="R0603" value="10k"/>
 <part name="SJ2" library="SparkFun" deviceset="SOLDERJUMPER" device="NO"/>
-<part name="C23" library="rcl" deviceset="C-EU" device="C0603" value="nc"/>
-<part name="R9" library="rcl" deviceset="R-EU_" device="R0805" value="nc"/>
 <part name="+3V10" library="supply1" deviceset="+3V3" device=""/>
 <part name="+3V11" library="supply1" deviceset="+3V3" device=""/>
@@
 <part name="R51" library="rcl" deviceset="R-EU_" device="R0603" value="nc"/>
 <part name="C92" library="rcl" deviceset="C-EU" device="C0603" value="10u"/>
-<part name="C93" library="rcl" deviceset="C-EU" device="C0603" value="100n"/>
 <part name="GND13" library="supply1" deviceset="GND" device=""/>
 <part name="SJ3" library="SparkFun" deviceset="SOLDERJUMPER" device="NO"/>
@@
 <part name="R12" library="rcl" deviceset="R-EU_" device="R0603" value="nc"/>
 <part name="P+1" library="supply1" deviceset="+5V" device=""/>
-<part name="S1" library="Mine" deviceset="TAC_SWITCH" device=""/>
 <part name="S2" library="Mine" deviceset="TAC_SWITCH" device=""/>
 <part name="S3" library="Mine" deviceset="TAC_SWITCH" device=""/>
@@
 <instance part="Q3" gate="G$1" x="25.4" y="-5.08" rot="R90"/>
 <instance part="SV4" gate="G$1" x="266.7" y="-27.94"/>
-<instance part="SV6" gate="G$1" x="287.02" y="-27.94"/>
 <instance part="IC12" gate="G$1" x="-40.64" y="147.32"/>
 <instance part="C28" gate="G$1" x="-55.88" y="139.7"/>
@@
 <instance part="D8" gate="G$1" x="-71.12" y="205.74"/>
 <instance part="D9" gate="G$1" x="-73.66" y="182.88"/>
-<instance part="L2" gate="G$1" x="-76.2" y="226.06" rot="R90"/>
 <instance part="C34" gate="G$1" x="-43.18" y="210.82"/>
 <instance part="GND9" gate="1" x="-43.18" y="203.2"/>
@@
 <instance part="R1" gate="G$1" x="-91.44" y="38.1"/>
 <instance part="SJ2" gate="1" x="137.16" y="-35.56"/>
-<instance part="C23" gate="G$1" x="-162.56" y="43.18" rot="R90"/>
-<instance part="R9" gate="G$1" x="-154.94" y="50.8" rot="R270"/>
 <instance part="+3V10" gate="G$1" x="-154.94" y="60.96"/>
 <instance part="+3V11" gate="G$1" x="93.98" y="-22.86"/>
@@
 <instance part="R51" gate="G$1" x="20.32" y="-7.62"/>
 <instance part="C92" gate="G$1" x="-104.14" y="17.78"/>
-<instance part="C93" gate="G$1" x="-96.52" y="68.58"/>
 <instance part="GND13" gate="1" x="-96.52" y="73.66" rot="R180"/>
 <instance part="SJ3" gate="1" x="-104.14" y="63.5"/>
@@
 <instance part="R12" gate="G$1" x="48.26" y="106.68" rot="R90"/>
 <instance part="P+1" gate="1" x="48.26" y="114.3"/>
-<instance part="S1" gate="S" x="-10.16" y="-27.94" rot="R270"/>
 <instance part="S2" gate="S" x="2.54" y="-27.94" rot="R270"/>
 <instance part="S3" gate="S" x="15.24" y="-27.94" rot="R270"/>
@@
 <wire x1="30.48" y1="48.26" x2="33.02" y2="48.26" width="0.1524" layer="91"/>
 </segment>
-<segment>
-<pinref part="C93" gate="G$1" pin="1"/>
-<pinref part="GND13" gate="1" pin="GND"/>
-</segment>
 </net>
 <net name="+5V" class="0">
@@
 <segment>
 <wire x1="294.64" y1="-30.48" x2="299.72" y2="-30.48" width="0.1524" layer="91"/>
-<pinref part="SV6" gate="G$1" pin="2"/>
 </segment>
 </net>
@@
 <segment>
 <wire x1="294.64" y1="-27.94" x2="299.72" y2="-27.94" width="0.1524" layer="91"/>
-<pinref part="SV6" gate="G$1" pin="3"/>
 </segment>
 </net>
@@
 <net name="VBAT" class="0">
 <segment>
-<wire x1="-86.36" y1="63.5" x2="-96.52" y2="63.5" width="0.1524" layer="91"/>
+<wire x1="-86.36" y1="63.5" x2="-99.06" y2="63.5" width="0.1524" layer="91"/>
 <label x="-93.98" y="63.5" size="1.778" layer="95"/>
 <pinref part="IC1" gate="G$1" pin="VBAT"/>
-<pinref part="C93" gate="G$1" pin="2"/>
-<wire x1="-96.52" y1="63.5" x2="-99.06" y2="63.5" width="0.1524" layer="91"/>
-<junction x="-96.52" y="63.5"/>
 <pinref part="SJ3" gate="1" pin="2"/>
 </segment>

Commit message: off for fab
Other:
- moved on the sheet: J2
Changed lines of the file:
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@@
 <instance part="SV1" gate="G$1" x="320.04" y="137.16"/>
 <instance part="SV2" gate="G$1" x="215.9" y="76.2"/>
-<instance part="J2" gate="G$1" x="-129.54" y="180.34"/>
+<instance part="J2" gate="G$1" x="-127" y="180.34"/>
 <instance part="C22" gate="G$1" x="-5.08" y="182.88"/>
 <instance part="Q3" gate="G$1" x="25.4" y="-5.08" rot="R90"/>
@@
 <segment>
 <wire x1="-116.84" y1="177.8" x2="-116.84" y2="172.72" width="0.1524" layer="91"/>
-<wire x1="-121.92" y1="180.34" x2="-116.84" y2="180.34" width="0.1524" layer="91"/>
+<wire x1="-119.38" y1="180.34" x2="-116.84" y2="180.34" width="0.1524" layer="91"/>
 <wire x1="-116.84" y1="180.34" x2="-116.84" y2="177.8" width="0.1524" layer="91"/>
-<wire x1="-116.84" y1="177.8" x2="-121.92" y2="177.8" width="0.1524" layer="91"/>
+<wire x1="-116.84" y1="177.8" x2="-119.38" y2="177.8" width="0.1524" layer="91"/>
 <junction x="-116.84" y="177.8"/>
 <pinref part="GND30" gate="1" pin="GND"/>
@@
 <pinref part="J2" gate="G$1" pin="4"/>
 <wire x1="-114.3" y1="182.88" x2="-91.44" y2="182.88" width="0.1524" layer="91"/>
-<wire x1="-119.38" y1="182.88" x2="-121.92" y2="182.88" width="0.1524" layer="91"/>
-</segment>
-</net>
+</segment>
+</net>
